File: EURORACK_PSU_3.kicad_sch (KiCad schematic)
At the start: 53 parts, among them J601 Eurorack_Power_16pin_Shrouded, J602 Eurorack_Power_16pin_Shrouded, Q601 MMBT2907*, Q602 MMBT2222A, Q603 MMBT2907*, U601 LM7812_TO220, U602 LM7912_TO220, U603 LM7805_TO220

Commit message: Misc
Connections:
- net +12v_out: now also J601.10 (GND), J601.9 (GND), J602.10 (GND), J602.9 (GND); no longer J601.7 (12V), J601.8 (+12V), J602.7 (12V), J602.8 (+12V)
- net +5v_out: now also J601.11 (GND), J601.12 (GND), J602.11 (GND), J602.12 (GND); no longer J601.5 (+12V), J601.6 (P6), J602.5 (+12V), J602.6 (P6)
- net -12v_out: now also J601.1 (P1), J601.2 (P2), J602.1 (P1), J602.2 (P2); no longer J601.15 (-12V), J601.16 (P16), J602.15 (-12V), J602.16 (P16)
- net GND: now also J601.3 (P3), J601.4 (P4), J601.5 (+12V), J601.6 (P6), J601.7 (12V), J601.8 (+12V), J602.3 (P3), J602.4 (P4), J602.5 (+12V), J602.6 (P6), J602.7 (12V), J602.8 (+12V); no longer J601.10 (GND), J601.11 (GND), J601.12 (GND), J601.13 (-12), J601.14 (-12V), J601.9 (GND), J602.10 (GND), J602.11 (GND), J602.12 (GND), J602.13 (-12), J602.14 (-12V), J602.9 (GND)
